Commit message: modified the urdf for the simulation on Gazebo

File: ROS/src/robot_description/urdf/robot.urdf.xacro (robot description, xacro)
@@ -1,4 +1,4 @@
 <?xml version="1.0"?>
-<robot xmlns:xacro="http://www.ros.org/wiki/xacro" name="firefighter">
+<robot xmlns:xacro="http://www.ros.org/wiki/xacro" name="Inverted_Pendulum">
 <xacro:property name="horizontal_ply_length" value="0.3"/>
 <xacro:property name="horizontal_ply_mass" value="0.1"/>
@@ -24,4 +24,7 @@
         </inertial>
 </xacro:macro>
+<material name="red">
+  <color rgba="0.8 0 0 1"/>
+</material>
     <link name="dummy_link">
     </link>
@@ -31,5 +34,6 @@
                 <box size="${horizontal_ply_length} ${ply_breadth} ${ply_thickness}"/>
             </geometry>
-            <origin xyz="0.0 0.0 ${ply_thickness/2+wheel_radius}" />
+            <material name="red"/>
+            <origin xyz="0.0 0.0 ${ply_thickness/2}" />
         </visual>
         <collision>
@@ -50,4 +54,5 @@
                 <box size="${vertical_ply_length} ${ply_breadth} ${ply_thickness}"/>
             </geometry>
+            <material name="red"/>
             <origin xyz="0.0 0.0 ${vertical_ply_length/2}" rpy="0.0 1.57075 0.0"/>
         </visual>
@@ -63,5 +68,5 @@
         <parent link="base_link"/>
         <child link="left_link"/>
-        <origin xyz="${horizontal_ply_length/2} 0.0 0.04"/>
+        <origin xyz="${horizontal_ply_length/2} 0.0 0.0"/>
     </joint>
     <link name="right_link">
@@ -70,4 +75,5 @@
                 <box size="${vertical_ply_length} ${ply_breadth} ${ply_thickness}"/>
             </geometry>
+            <material name="red"/>
             <origin xyz="0.0 0.0 ${vertical_ply_length/2}" rpy="0.0 1.57075 0.0"/>
         </visual>
@@ -82,5 +88,5 @@
         <parent link="base_link"/>
         <child link="right_link"/>
-        <origin xyz="${-horizontal_ply_length/2} 0.0 0.04" />
+        <origin xyz="${-horizontal_ply_length/2} 0.0 0.0" />
     </joint>
     <link name="top_link">
@@ -89,4 +95,5 @@
                 <box size="${horizontal_ply_length} ${ply_breadth} ${ply_thickness}"/>
             </geometry>
+            <material name="red"/>
             <origin xyz="0.0 0.0 ${-ply_thickness/2}" />
         </visual>
@@ -114,4 +121,5 @@
                 <box size="${horizontal_ply_length} ${ply_breadth} ${ply_thickness}"/>
             </geometry>
+            <material name="red"/>
             <origin xyz="${-horizontal_ply_length/2} 0.0 0.01" />
         </visual>
@@ -139,4 +147,5 @@
                 <cylinder radius="${wheel_radius}" length="${wheel_thickness}"/>
             </geometry>
+            <material name="red"/>
             <origin rpy="0.0 1.57075 0.0"/>
         </visual>
@@ -153,5 +162,5 @@
         <parent link="base_link"/>
         <child link="left_wheel"/>
-        <origin xyz="0.18 0.0 0.04" />
+        <origin xyz="0.18 0.0 0.0" />
     </joint>
     <link name="right_wheel">
@@ -160,4 +169,5 @@
                 <cylinder radius="${wheel_radius}" length="${wheel_thickness}"/>
             </geometry>
+            <material name="red"/>
             <origin rpy="0.0 1.57075 0.0"/>
         </visual>
@@ -173,5 +183,5 @@
         <parent link="base_link"/>
         <child link="right_wheel"/>
-        <origin xyz="-0.18 0.0 0.04" />
+        <origin xyz="-0.18 0.0 0.0" />
     </joint>
     <link name="imu_link">
@@ -182,3 +192,4 @@
         <origin xyz="0.01 0.0 0.0" />
     </joint>
+    <xacro:include filename="robot.gazebo.xacro"/>
 </robot>
